Commit message: Working with PID Controller Output

File: thesis_arm/urdf/thesis_arm.urdf (robot description, URDF)
Before this commit: robot thesis_arm, 7 links, 6 joints
Joints:
- joint Joint_1: limit lower=-2.79253 upper=2.79253 effort=255 velocity=0 -> lower=-2.79253 upper=2.79253 effort=1 velocity=0
- joint Joint_2: limit lower=-1.5708 upper=1.5708 effort=255 velocity=0 -> lower=-1.5708 upper=1.5708 effort=1 velocity=0
- joint Joint_3: limit lower=-3.14159 upper=0.872665 effort=255 velocity=0 -> lower=-3.14159 upper=0.872665 effort=1 velocity=0
- joint Joint_4: limit lower=-3.14159 upper=3.14159 effort=255 velocity=0 -> lower=-3.14159 upper=3.14159 effort=1 velocity=0
- joint Joint_5: limit lower=-1.5708 upper=1.5708 effort=255 velocity=0 -> lower=-1.5708 upper=1.5708 effort=1 velocity=0
- joint Joint_6: limit lower=-3.14159 upper=3.14159 effort=255 velocity=0 -> lower=-3.14159 upper=3.14159 effort=1 velocity=0

Commit message: Updated with joint 5 and velocity and acceleration

File: thesis_arm/urdf/thesis_arm.urdf (robot description, URDF)
Before this commit: robot thesis_arm, 7 links, 6 joints
Joints:
- joint Joint_3: limit lower=-3.14159 upper=0.872665 effort=1 velocity=0 -> lower=-3.14159 upper=3.14159 effort=1 velocity=0
