Commit message: Updated hardware Controller
Updated Python Script for position control
Updated Launch file and RViz config

File: bcr1_description/urdf/bcr1_description.urdf (robot description, URDF)
Before this commit: robot bcr1_description, 7 links, 6 joints
Joints:
- joint Joint_5: limit lower=-2.26893 upper=2.26893 effort=0 velocity=0 -> lower=-1.5708 upper=1.5708 effort=0 velocity=0
